Commit message: add a start program and an example, while fr5 doesn't work

File: assets/urdf/fr5_robot_descripiton/robots/fr5_robot.urdf (robot description, URDF)
Before this commit: robot fr5_robot, 8 links, 7 joints
Links:
- link base_link: geometry collision mesh filename=/home/lhc/PycharmProjects/Comprehensive-design-of-intellige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; visual mesh filename=/home/lhc/PycharmProjects/Comprehensive-design-of-intellige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
- link forearm_Link: geometry collision mesh filename=/home/lhc/PycharmProjects/Comprehensive-design-of-intellige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; visual mesh filename=/home/lhc/PycharmProjects/Comprehensive-design-of-intellige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
- link shoulder_Link: geometry collision mesh filename=/home/lhc/PycharmProjects/Comprehensive-design-of-intellige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; visual mesh filename=/home/lhc/PycharmProjects/Comprehensive-design-of-intellige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
- link upperarm_Link: geometry collision mesh filename=/home/lhc/PycharmProjects/Comprehensive-design-of-intellige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; visual mesh filename=/home/lhc/PycharmProjects/Comprehensive-design-of-intellige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
- link wrist1_Link: geometry collision mesh filename=/home/lhc/PycharmProjects/Comprehensive-design-of-intellige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; visual mesh filename=/home/lhc/PycharmProjects/Comprehensive-design-of-intellige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
- link wrist2_Link: geometry collision mesh filename=/home/lhc/PycharmProjects/Comprehensive-design-of-intellige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; visual mesh filename=/home/lhc/PycharmProjects/Comprehensive-design-of-intellige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
- link wrist3_Link: geometry collision mesh filename=/home/lhc/PycharmProjects/Comprehensive-design-of-intellige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; visual mesh filename=/home/lhc/PycharmProjects/Comprehensive-design-of-intellige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

Commit message: fix fr5 urdf parsing wrong

File: assets/urdf/fr5_robot_descripiton/robots/fr5_robot.urdf (robot description, URDF)
Before this commit: robot fr5_robot, 8 links, 7 joints
Links:
- removed link world
- link base_link: geometry collision mesh filename=../meshes/collision/base_link.STL; visual mesh filename=../meshes/visual/base.dae
- link forearm_Link: geometry collision mesh filename=../meshes/collision/forearm_Link.STL; visual mesh filename=../meshes/visual/forearm.dae
- link shoulder_Link: geometry collision mesh filename=../meshes/collision/shoulder_Link.STL; visual mesh filename=../meshes/visual/shoulder.dae
- link upperarm_Link: geometry collision mesh filename=../meshes/collision/upperarm_Link.STL; visual mesh filename=../meshes/visual/upperarm.dae
- link wrist1_Link: geometry collision mesh filename=../meshes/collision/wrist1_Link.STL; visual mesh filename=../meshes/visual/wrist1.dae
- link wrist2_Link: geometry collision mesh filename=../meshes/collision/wrist2_Link.STL; visual mesh filename=../meshes/visual/wrist2.dae
- link wrist3_Link: geometry collision mesh filename=../meshes/collision/wrist3_Link.STL; visual mesh filename=../meshes/visual/wrist3.dae
Joints:
- removed joint world
